File: Lilypad buffered/Lilypad buffered.brd (EAGLE design)
At the start: 50 x 50 mm, 45 parts, among them T1 MMBTA3904, T10 MMBTA3904, T11 MMBTA3906, T12 MMBTA3904, T13 MMBTA3906, T14 MMBTA3904, T15 MMBTA3906, T16 MMBTA3904, T2 MMBTA3906, T3 MMBTA3906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

Commit message: Cambiado el formato de las perforaciones de Excellon a gerber-RS274X. - Actualizados los gerber involucrados. - Actualizado archivo cam involucrado. - Mejoras menores a la tarjeta de Lilypad con bufferes.
Parts:
- removed JP1: (no value), pinhead:2X03
- removed R13, R14, R15, R16: 470, resistor:R0603
- removed T13, T15: MMBTA3906, transistor:SOT23-BEC
- removed T14, T16: MMBTA3904, transistor-neu-to92:SOT23-BEC
- removed U$7: 7, LilyPad-Wearables:PETAL-LONG-1-2SIDE
- removed U$8: 8, LilyPad-Wearables:PETAL-LONG-1-2SIDE
- added C1: (no value), rcl:C0603
- added J1: AVR_SPI_PRG_6PTH, SparkFun-Connectors:2X3
- added J2: (no value), SparkFun-Connectors:JST-2-SMD
- added U2: MIC5219-3.3BM5, SparkFun-PowerIC:SOT23-5
Connections:
- removed net N$31: T13.C, T14.C, U$7.1
- removed net N$32: R13.1
- removed net N$33: R14.1
- removed net N$34: R16.2, T16.B
- removed net N$35: R15.2, T15.B
- removed net N$36: T15.C, T16.C, U$8.1
- removed net N$37: R15.1
- removed net N$38: R16.1
- net +3V3: no longer T13.E, T15.E
- net GND: now also C1.2, J2.1, U2.2; no longer T14.E, T16.E
- net N$29: now also C1.1, U2.4; no longer R14.2, T14.B
- net N$30: now also J2.2, U2.1; no longer R13.2, T13.B
Changed lines of the file:
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@@
 <element name="R12" library="resistor" package="R0603" value="470" x="-26.67" y="53.34"/>
 <element name="U$6" library="LilyPad-Wearables" package="PETAL-LONG-1-2SIDE" value="6" x="33.02" y="41.91" rot="R270"/>
-<element name="JP1" library="pinhead" package="2X03" value="" x="-8.89" y="30.48" rot="R90"/>
-<element name="T13" library="transistor" package="SOT23-BEC" value="MMBTA3906" x="-52.07" y="10.16"/>
-<element name="R13" library="resistor" package="R0603" value="470" x="-59.69" y="10.16"/>
-<element name="T14" library="transistor-neu-to92" package="SOT23-BEC" value="MMBTA3904" x="-52.07" y="3.81"/>
-<element name="R14" library="resistor" package="R0603" value="470" x="-64.77" y="31.75"/>
-<element name="U$7" library="LilyPad-Wearables" package="PETAL-LONG-1-2SIDE" value="7" x="3.81" y="13.97"/>
-<element name="T15" library="transistor" package="SOT23-BEC" value="MMBTA3906" x="-63.5" y="24.13"/>
-<element name="R15" library="resistor" package="R0603" value="470" x="-66.04" y="13.97"/>
-<element name="T16" library="transistor-neu-to92" package="SOT23-BEC" value="MMBTA3904" x="-58.42" y="20.32"/>
-<element name="R16" library="resistor" package="R0603" value="470" x="-71.12" y="3.81"/>
-<element name="U$8" library="LilyPad-Wearables" package="PETAL-LONG-1-2SIDE" value="8" x="36.83" y="12.7" rot="R180"/>
 <element name="U$9" library="LilyPad-Wearables" package="PETAL-LONG-1-2SIDE" value="+" x="10.16" y="46.99"/>
 <element name="U$10" library="LilyPad-Wearables" package="PETAL-LONG-1-2SIDE" value="-" x="27.94" y="46.99" rot="R180"/>
 <element name="U$11" library="LilyPad-Wearables" package="PETAL-LONG-1-2SIDE" value="+" x="-68.58" y="-2.54"/>
+<element name="J1" library="SparkFun-Connectors" package="2X3" value="AVR_SPI_PRG_6PTH" x="-78.74" y="-1.27"/>
+<element name="J2" library="SparkFun-Connectors" package="JST-2-SMD" value="" x="-85.09" y="1.27">
+<attribute name="PROD_ID" value="CONN-08352" x="-85.09" y="1.27" size="1.778" layer="27" display="off"/>
+</element>
+<element name="U2" library="SparkFun-PowerIC" package="SOT23-5" value="MIC5219-3.3BM5" x="-91.44" y="-2.54">
+<attribute name="PROD_ID" value="VREG-00822" x="-91.44" y="-2.54" size="1.778" layer="27" display="off"/>
+</element>
+<element name="C1" library="rcl" package="C0603" value="" x="-91.44" y="-7.62"/>
 </elements>
 <signals>
@@
 <contactref element="T10" pad="E"/>
 <contactref element="T12" pad="E"/>
-<contactref element="T14" pad="E"/>
-<contactref element="T16" pad="E"/>
 <contactref element="U$10" pad="1"/>
-<wire x1="-51.12" y1="2.71" x2="27.91" y2="46.99" width="0" layer="19" extent="1-1"/>
-<wire x1="-57.47" y1="19.22" x2="-51.12" y2="2.71" width="0" layer="19" extent="1-1"/>
-<wire x1="-47.31" y1="24.3" x2="-57.47" y2="19.22" width="0" layer="19" extent="1-1"/>
+<contactref element="C1" pad="2"/>
+<contactref element="U2" pad="2"/>
+<contactref element="J2" pad="1"/>
+<wire x1="-91.44" y1="-3.8401" x2="-90.59" y2="-7.62" width="0" layer="19" extent="1-1"/>
+<wire x1="-86.09" y1="-2.43" x2="-91.44" y2="-3.8401" width="0" layer="19" extent="1-1"/>
+<wire x1="-47.31" y1="24.3" x2="-86.09" y2="-2.43" width="0" layer="19" extent="1-1"/>
 <wire x1="-34.61" y1="16.68" x2="-47.31" y2="24.3" width="0" layer="19" extent="1-1"/>
 <wire x1="-21.91" y1="24.3" x2="-34.61" y2="16.68" width="0" layer="19" extent="1-1"/>
@@
 <wire x1="-19.37" y1="40.81" x2="-21.91" y2="24.3" width="0" layer="19" extent="1-1"/>
 <wire x1="18.1" y1="13.8" x2="-21.91" y2="24.3" width="0" layer="19" extent="1-1"/>
+<wire x1="27.91" y1="46.99" x2="18.1" y2="13.8" width="0" layer="19" extent="1-1"/>
 </signal>
 <signal name="+3V3">
@@
 <contactref element="T9" pad="E"/>
 <contactref element="T11" pad="E"/>
-<contactref element="T13" pad="E"/>
-<contactref element="T15" pad="E"/>
 <contactref element="U$9" pad="1"/>
-<wire x1="-51.12" y1="9.06" x2="10.19" y2="46.99" width="0" layer="19" extent="1-1"/>
-<wire x1="-47.31" y1="16.68" x2="-51.12" y2="9.06" width="0" layer="19" extent="1-1"/>
-<wire x1="-34.61" y1="24.3" x2="-47.31" y2="16.68" width="0" layer="19" extent="1-1"/>
+<wire x1="21.91" y1="13.8" x2="10.19" y2="46.99" width="0" layer="19" extent="1-1"/>
+<wire x1="-21.91" y1="31.92" x2="10.19" y2="46.99" width="0" layer="19" extent="1-1"/>
+<wire x1="-34.61" y1="24.3" x2="-21.91" y2="31.92" width="0" layer="19" extent="1-1"/>
+<wire x1="-47.31" y1="16.68" x2="-34.61" y2="24.3" width="0" layer="19" extent="1-1"/>
 <wire x1="-47.31" y1="31.92" x2="-34.61" y2="24.3" width="0" layer="19" extent="1-1"/>
-<wire x1="-21.91" y1="31.92" x2="-34.61" y2="24.3" width="0" layer="19" extent="1-1"/>
 <wire x1="-21.91" y1="16.68" x2="-34.61" y2="24.3" width="0" layer="19" extent="1-1"/>
-<wire x1="-62.55" y1="23.03" x2="-47.31" y2="16.68" width="0" layer="19" extent="1-1"/>
-<wire x1="21.91" y1="13.8" x2="-21.91" y2="16.68" width="0" layer="19" extent="1-1"/>
 </signal>
 <signal name="N$4">
@@
 </signal>
 <signal name="N$29">
-<contactref element="R14" pad="2"/>
-<contactref element="T14" pad="B"/>
-<wire x1="-63.92" y1="31.75" x2="-53.02" y2="2.71" width="0" layer="19" extent="1-1"/>
+<contactref element="U2" pad="4"/>
+<contactref element="C1" pad="1"/>
+<wire x1="-90.49" y1="-1.2399" x2="-92.29" y2="-7.62" width="0" layer="19" extent="1-1"/>
 </signal>
 <signal name="N$30">
-<contactref element="T13" pad="B"/>
-<contactref element="R13" pad="2"/>
-<wire x1="-53.02" y1="9.06" x2="-58.84" y2="10.16" width="0" layer="19" extent="1-1"/>
-</signal>
-<signal name="N$31">
-<contactref element="T13" pad="C"/>
-<contactref element="T14" pad="C"/>
-<contactref element="U$7" pad="1"/>
-<wire x1="-52.07" y1="11.26" x2="-52.07" y2="4.91" width="0" layer="19" extent="1-1"/>
-<wire x1="3.84" y1="13.97" x2="-52.07" y2="11.26" width="0" layer="19" extent="1-1"/>
-</signal>
-<signal name="N$32">
-<contactref element="R13" pad="1"/>
-</signal>
-<signal name="N$33">
-<contactref element="R14" pad="1"/>
-</signal>
-<signal name="N$34">
-<contactref element="R16" pad="2"/>
-<contactref element="T16" pad="B"/>
-<wire x1="-59.37" y1="19.22" x2="-70.27" y2="3.81" width="0" layer="19" extent="1-1"/>
-</signal>
-<signal name="N$35">
-<contactref element="T15" pad="B"/>
-<contactref element="R15" pad="2"/>
-<wire x1="-64.45" y1="23.03" x2="-65.19" y2="13.97" width="0" layer="19" extent="1-1"/>
-</signal>
-<signal name="N$36">
-<contactref element="T15" pad="C"/>
-<contactref element="T16" pad="C"/>
-<contactref element="U$8" pad="1"/>
-<wire x1="-58.42" y1="21.42" x2="36.8" y2="12.7" width="0" layer="19" extent="1-1"/>
-<wire x1="-63.5" y1="25.23" x2="-58.42" y2="21.42" width="0" layer="19" extent="1-1"/>
-</signal>
-<signal name="N$37">
-<contactref element="R15" pad="1"/>
-</signal>
-<signal name="N$38">
-<contactref element="R16" pad="1"/>
+<contactref element="U2" pad="1"/>
+<contactref element="J2" pad="2"/>
+<wire x1="-84.09" y1="-2.43" x2="-92.39" y2="-3.8401" width="0" layer="19" extent="1-1"/>
 </signal>
 </signals>

Commit message: Continuado el trabajo sobre el esquematico. Terminado sistema minimo y fuente de suministro (con proteccion).
Parts:
- removed U$11: +, LilyPad-Wearables:PETAL-LONG-1-2SIDE
- added C2, C3: 100nF, rcl:C0805K
- added F1: PTC 500mA, Personal - Varios:SMD-2012
- added R13: 10K, resistor:R0603
- C1: value (none) -> 10nF; device rcl:C0603 -> rcl:C0805K
- moved U$3 40.2 mm to (19.1, -5.08)
- moved U$4 38.4 mm to (17.8, 1.27)
- moved U$9 37.4 mm to (-11.4, 16.5)
- moved J2 36.6 mm to (-97.8, -33.0)
- moved U$10 36.0 mm to (3.81, 20.3)
- moved U1 34.5 mm to (0.00, 0.00)
- moved U$6 34.2 mm to (15.2, 12.7)
- moved U$5 33.8 mm to (-20.3, 0.00)
- moved U$2 33.5 mm to (-19.1, 8.89)
- moved U$1 32.1 mm to (2.54, -20.3)
- moved R1 30.6 mm to (3.81, 39.4)
- moved T2 29.6 mm to (2.54, 34.3)
- moved R2 25.7 mm to (6.35, 38.1)
- moved T1 19.7 mm to (14.0, 31.8)
Connections:
- new net N$31: J1.3, U1.17
- new net N$32: J1.1, U1.16
- new net N$33: J1.4, U1.15
- new net N$34: C3.1, R13.1, U1.29
- new net N$35: F1.P$1, U2.1
- new net N$36: C3.2, J1.5
- net +3V3: now also C2.1, J1.2, R13.2, U1.18, U1.4, U1.6, U2.5
- net GND: now also C2.2, J1.6, U1.21, U1.3, U1.5, U2.3
- net N$30: now also F1.P$2; no longer U2.1
